File: hardware/SBK_SP1.kicad_pcb (KiCad board)
At the start: 2 copper layers, 10.7 x 11.1 mm, 10 parts, among them J1 1x4 pin header, Q1 AO3400A, Q2 AO3401A

Commit message: updates
Other:
- board text added: "SBK_SP1 v1.0"
- board text removed: "SBK SP1 v1.0"

Commit message: KiCad files update
Connections:
- net Net-(J1-Pin_4) renamed CTRL
Changed lines of the file:
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@@
 			)
 		)
-		(property "Description" "P-channel MOSFET"
+		(property "Description" "N-channel MOSFET"
 			(at 0 0 0)
 			(layer "F.Fab")
@@
 			(pinfunction "S_2")
 			(pintype "passive")
+			(thermal_gap 0.2)
 		)
 		(pad "3" smd roundrect
@@
 			(layers "F.Cu" "F.Mask" "F.Paste")
 			(roundrect_rratio 0.25)
-			(net "Net-(J1-Pin_4)")
+			(net "CTRL")
 			(pintype "passive")
 		)
@@
 			(net "GND")
 			(pintype "passive")
+			(thermal_bridge_width 0.6)
+			(thermal_gap 0.2)
 		)
 		(embedded_fonts no)
@@
 			)
 		)
-		(property "Description" "N-channel MOSFET"
+		(property "Description" "P-channel MOSFET"
 			(at 0 0 0)
 			(layer "F.Fab")
@@
 			(layers "*.Cu" "*.Mask")
 			(remove_unused_layers no)
-			(net "Net-(J1-Pin_4)")
+			(net "CTRL")
 			(pinfunction "Pin_4_4")
 			(pintype "passive")
@@
 		(width 0.4)
 		(layer "F.Cu")
-		(net "Net-(J1-Pin_4)")
+		(net "CTRL")
 	)
 	(segment
@@
 		(width 0.4)
 		(layer "F.Cu")
-		(net "Net-(J1-Pin_4)")
+		(net "CTRL")
 	)
 	(segment
@@
 		(width 0.4)
 		(layer "F.Cu")
-		(net "Net-(J1-Pin_4)")
+		(net "CTRL")
 	)
 	(segment
@@
 		(width 0.4)
 		(layer "F.Cu")
-		(net "Net-(J1-Pin_4)")
+		(net "CTRL")
 	)
 	(segment
@@
 		(width 0.4)
 		(layer "F.Cu")
-		(net "Net-(J1-Pin_4)")
+		(net "CTRL")
 	)
 	(zone
@@
 		(hatch edge 0.5)
 		(connect_pads
-			(clearance 0.25)
+			(clearance 0.2)
 		)
 		(min_thickness 0.25)
