File: hardware/SBK_SP1.kicad_sch (KiCad schematic)
At the start: 10 parts, among them J1 1x4 pin header, Q1 AO3400A, Q2 AO3401A

Commit message: KiCad files update
Connections:
- net CTRL: now reaches J1.4 (Pin_4), R1.2
Changed lines of the file:
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@@
+	)
+	(junction
+		(at 77.47 140.335)
+		(diameter 0)
+		(color 0 0 0 0)
 	)
 	(junction
@@
 	(wire
 		(pts
+			(xy 77.47 144.78) (xy 77.47 140.335)
+		)
+		(stroke
+			(width 0)
+			(type default)
+		)
+	)
+	(wire
+		(pts
 			(xy 79.375 135.255) (xy 79.375 153.67)
 		)
@@
 	(wire
 		(pts
+			(xy 73.66 144.78) (xy 77.47 144.78)
+		)
+		(stroke
+			(width 0)
+			(type default)
+		)
+	)
+	(wire
+		(pts
 			(xy 83.82 137.795) (xy 83.82 149.225)
 		)
@@
 			(width 0)
 			(type default)
+		)
+	)
+	(global_label "CTRL"
+		(shape input)
+		(at 73.66 144.78 180)
+		(fields_autoplaced yes)
+		(effects
+			(font
+				(size 1.27 1.27)
+			)
+			(justify right)
+		)
+		(property "Intersheetrefs" "${INTERSHEET_REFS}"
+			(at 66.1391 144.78 0)
+			(hide yes)
+			(show_name no)
+			(do_not_autoplace no)
+			(effects
+				(font
+					(size 1.27 1.27)
+				)
+				(justify right)
+			)
 		)
 	)
@@
 			)
 		)
-		(property "Description" "P-channel MOSFET"
+		(property "Description" "N-channel MOSFET"
 			(at 105.41 140.335 0)
 			(hide yes)
@@
 			)
 		)
-		(property "Description" "N-channel MOSFET"
+		(property "Description" "P-channel MOSFET"
 			(at 114.935 130.175 0)
 			(hide yes)
